File: SSA_LED_Board_1/SSA_LED_Board_1.kicad_sch (KiCad schematic)
At the start: 36 parts, among them J1 EJ508A, U1 BCR401U, U2 BCR401U

Commit message: finished layout
Parts:
- removed J1: EJ508A, EJ508A:MPD_EJ508A, symbol EJ508A:EJ508A
- added H1, H2, H3: MountingHole, MountingHole:MountingHole_2.2mm_M2, symbol Mechanical:MountingHole
- added J1: 54-00164, 54-00164:TENSILITY_54-00164, symbol 54-00164:54-00164
Connections:
- net GND: now also J1.B, J1.C
- net Power_in: now also J1.A1, J1.A2
